File: Boost.sch (KiCad schematic (older format))
At the start: 23 parts, among them Q1 IRFZ44N, U1 UC3843_DIP8

Commit message: Reducción de placa
Se redujo la placa de 10cm x 20cm a 5cm x 10 cm.
Parts:
- COUT1: footprint Capacitor_THT:CP_Radial_D25.0mm_P10.00mm_SnapIn -> Capacitor_THT:CP_Radial_D8.0mm_P5.00mm
- L1: footprint Inductor_THT:Choke_EPCOS_B82722A -> Inductor_THT:L_Axial_L9.5mm_D4.0mm_P15.24mm_Horizontal_Fastron_SMCC
Changed lines of the file:
@@
 F 0 "L1" H 7952 2696 50  0000 L CNN
 F 1 "200u" H 7952 2605 50  0000 L CNN
-F 2 "Inductor_THT:Choke_EPCOS_B82722A" H 7900 2650 50  0001 C CNN
+F 2 "Inductor_THT:L_Axial_L9.5mm_D4.0mm_P15.24mm_Horizontal_Fastron_SMCC" H 7900 2650 50  0001 C CNN
 F 3 "~" H 7900 2650 50  0001 C CNN
 	1    7900 2650
@@
 F 0 "COUT1" H 9018 3246 50  0000 L CNN
 F 1 "100u" H 9018 3155 50  0000 L CNN
-F 2 "Capacitor_THT:CP_Radial_D25.0mm_P10.00mm_SnapIn" H 8938 3050 50  0001 C CNN
+F 2 "Capacitor_THT:CP_Radial_D8.0mm_P5.00mm" H 8938 3050 50  0001 C CNN
 F 3 "~" H 8900 3200 50  0001 C CNN
 	1    8900 3200
