File: Boost.kicad_pcb (KiCad board)
At the start: 2 copper layers, 32 parts, among them Q1 IRFZ24N, U1 UC3843_DIP8

Commit message: Disipador + Bobina.
Parts:
- L1: footprint Inductor_THT:L_Axial_L9.5mm_D4.0mm_P15.24mm_Horizontal_Fastron_SMCC -> Inductor_THT:Inductor_26mm_x_8mm
- moved L1 14.8 mm to (127.8, 49.0), turned to 0 degrees
Routing:
- net +15V: track 125.7 -> 110.7 mm
- net Net-(JPl1-Pad2): track 31.7 -> 21.2 mm
- net Net-(DOUT1-Pad1): track 79.1 -> 84.2 mm
- net (no net): vias 0 -> 2
Changed lines of the file:
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@@
-(kicad_pcb (version 20171130) (host pcbnew "(5.1.0)-1")
+(kicad_pcb (version 20171130) (host pcbnew "(5.1.2)-1")
   (general
     (thickness 1.6)
-    (drawings 8)
-    (tracks 159)
+    (drawings 12)
+    (tracks 165)
     (zones 0)
     (modules 32)
@@
   )
   (setup
-    (last_trace_width 2)
+    (last_trace_width 4)
     (user_trace_width 1)
     (user_trace_width 2)
@@
     (add_net "Net-(RG1-Pad2)")
     (add_net "Net-(ROSC1-Pad1)")
+  )
+  (module Inductor_THT:Inductor_26mm_x_8mm (layer F.Cu)
+    (at 127.75 49)
+    (fp_text reference L1 (at 13.54 -3.85) (layer F.SilkS)
+      (effects (font (size 1 1) (thickness 0.15)))
+    )
+    (fp_text value 200u (at 13.54 -4.85) (layer F.Fab)
+      (effects (font (size 1 1) (thickness 0.15)))
+    )
+    (fp_line (start -1 1) (end -1 -9) (layer F.SilkS) (width 0.12))
+    (fp_line (start 27 1) (end -1 1) (layer F.SilkS) (width 0.12))
+    (fp_line (start 27 -9) (end 27 1) (layer F.SilkS) (width 0.12))
+    (fp_line (start -1 -9) (end 27 -9) (layer F.SilkS) (width 0.12))
+    (pad 4 thru_hole circle (at 26 -8) (size 1.524 1.524) (drill 0.762) (layers *.Cu *.Mask))
+    (pad 3 thru_hole circle (at 0 -8) (size 1.524 1.524) (drill 0.762) (layers *.Cu *.Mask))
+    (pad 2 thru_hole circle (at 26 0) (size 1.524 1.524) (drill 0.762) (layers *.Cu *.Mask)
+      (net 16 "Net-(JPl1-Pad2)"))
+    (pad 1 thru_hole rect (at 0 0) (size 1.524 1.524) (drill 0.762) (layers *.Cu *.Mask)
+      (net 1 +15V))
   )
   (module Connector:Banana_Jack_1Pin (layer F.Cu)
@@
     )
   )
-  (module Inductor_THT:L_Axial_L9.5mm_D4.0mm_P15.24mm_Horizontal_Fastron_SMCC (layer F.Cu)
-    (at 142.5 49 90)
-    (descr "Inductor, Axial series, Axial, Horizontal, pin pitch=15.24mm, , length*diameter=9.5*4mm^2, Fastron, SMCC, http://cdn-reichelt.de/documents/datenblatt/B400/DS_SMCC_NEU.pdf, http://cdn-reichelt.de/documents/datenblatt/B400/LEADEDINDUCTORS.pdf")
-    (tags "Inductor Axial series Axial Horizontal pin pitch 15.24mm  length 9.5mm diameter 4mm Fastron SMCC")
-    (fp_text reference L1 (at 7.62 -3.12 90) (layer F.SilkS)
-      (effects (font (size 1 1) (thickness 0.15)))
-    )
-    (fp_text value 200u (at 7.62 3.12 90) (layer F.Fab)
-      (effects (font (size 1 1) (thickness 0.15)))
-    )
-    (fp_text user %R (at 7.62 0 90) (layer F.Fab)
-      (effects (font (size 1 1) (thickness 0.15)))
-    )
-    (fp_line (start 16.5 -2.25) (end -1.25 -2.25) (layer F.CrtYd) (width 0.05))
-    (fp_line (start 16.5 2.25) (end 16.5 -2.25) (layer F.CrtYd) (width 0.05))
-    (fp_line (start -1.25 2.25) (end 16.5 2.25) (layer F.CrtYd) (width 0.05))
-    (fp_line (start -1.25 -2.25) (end -1.25 2.25) (layer F.CrtYd) (width 0.05))
-    (fp_line (start 14 0) (end 12.49 0) (layer F.SilkS) (width 0.12))
-    (fp_line (start 1.24 0) (end 2.75 0) (layer F.SilkS) (width 0.12))
-    (fp_line (start 12.49 -2.12) (end 2.75 -2.12) (layer F.SilkS) (width 0.12))
-    (fp_line (start 12.49 2.12) (end 12.49 -2.12) (layer F.SilkS) (width 0.12))
-    (fp_line (start 2.75 2.12) (end 12.49 2.12) (layer F.SilkS) (width 0.12))
-    (fp_line (start 2.75 -2.12) (end 2.75 2.12) (layer F.SilkS) (width 0.12))
-    (fp_line (start 15.24 0) (end 12.37 0) (layer F.Fab) (width 0.1))
-    (fp_line (start 0 0) (end 2.87 0) (layer F.Fab) (width 0.1))
-    (fp_line (start 12.37 -2) (end 2.87 -2) (layer F.Fab) (width 0.1))
-    (fp_line (start 12.37 2) (end 12.37 -2) (layer F.Fab) (width 0.1))
-    (fp_line (start 2.87 2) (end 12.37 2) (layer F.Fab) (width 0.1))
-    (fp_line (start 2.87 -2) (end 2.87 2) (layer F.Fab) (width 0.1))
-    (pad 2 thru_hole oval (at 15.24 0 90) (size 2 2) (drill 1) (layers *.Cu *.Mask)
-      (net 16 "Net-(JPl1-Pad2)"))
-    (pad 1 thru_hole circle (at 0 0 90) (size 2 2) (drill 1) (layers *.Cu *.Mask)
-      (net 1 +15V))
-    (model ${KISYS3DMOD}/Inductor_THT.3dshapes/L_Axial_L9.5mm_D4.0mm_P15.24mm_Horizontal_Fastron_SMCC.wrl
-      (at (xyz 0 0 0))
-      (scale (xyz 1 1 1))
-      (rotate (xyz 0 0 0))
-    )
-  )
   (module Potentiometer_THT:Potentiometer_Bourns_3266Y_Vertical (layer F.Cu)
     (at 173.44148 102.6461 90)
@@
     )
   )
+  (gr_line (start 155.025 92.275) (end 179.025 92.275) (layer F.SilkS) (width 0.12))
+  (gr_line (start 167.025 92.275) (end 155.025 92.275) (layer F.SilkS) (width 0.12))
+  (gr_line (start 167.025 91.775) (end 167.025 92.275) (layer F.SilkS) (width 0.12))
+  (gr_line (start 167.025 88.375) (end 167.025 91.775) (layer F.SilkS) (width 0.12))
   (gr_circle (center 195 125) (end 196.5 125) (layer F.SilkS) (width 0.12))
   (gr_circle (center 195 35) (end 196.5 35) (layer F.SilkS) (width 0.12))
@@
   (gr_line (start 200 130) (end 200 30) (layer F.Adhes) (width 0.15))
   (gr_line (start 100 130) (end 200 130) (layer F.Adhes) (width 0.15))
+  (via (at 179.025 92.275) (size 2) (drill 1) (layers F.Cu B.Cu) (net 0))
+  (via (at 155.025 92.275) (size 2) (drill 1) (layers F.Cu B.Cu) (net 0))
   (segment (start 113 43) (end 119 49) (width 4) (layer B.Cu) (net 1))
   (segment (start 119 49) (end 113 55) (width 1) (layer B.Cu) (net 1))
@@
   (segment (start 152.5 72.75) (end 147.25 67.5) (width 1) (layer B.Cu) (net 1))
   (segment (start 152.5 73) (end 152.5 72.75) (width 1) (layer B.Cu) (net 1))
-  (segment (start 119 49) (end 142.75 49) (width 4) (layer B.Cu) (net 1))
   (segment (start 120 79.5) (end 122.5 79.5) (width 1) (layer B.Cu) (net 1))
   (segment (start 113 55) (end 113 72.5) (width 1) (layer B.Cu) (net 1))
   (segment (start 113 72.5) (end 120 79.5) (width 1) (layer B.Cu) (net 1))
+  (segment (start 119 49) (end 127.75 49) (width 4) (layer B.Cu) (net 1))
   (segment (start 154.0689 111.54626) (end 154.08668 111.56404) (width 2) (layer B.Cu) (net 2))
   (segment (start 113 117) (end 120.184204 117) (width 4) (layer B.Cu) (net 2))
@@
   (segment (start 180.5 60.96) (end 179.297919 60.96) (width 1) (layer B.Cu) (net 14))
   (segment (start 178 98) (end 173.5 102.5) (width 1) (layer B.Cu) (net 14))
-  (segment (start 178 62.5) (end 178 98) (width 1) (layer B.Cu) (net 14))
   (segment (start 181.25 48.75) (end 187 43) (width 2) (layer B.Cu) (net 14))
   (segment (start 181.25 53.25) (end 181.25 48.75) (width 2) (layer B.Cu) (net 14))
@@
   (segment (start 181.25 53.25) (end 185.36 57.36) (width 2) (layer B.Cu) (net 14))
   (segment (start 185.36 57.36) (end 185.36 57.64) (width 2) (layer B.Cu) (net 14))
+  (segment (start 178 98) (end 180.55 98) (width 1) (layer B.Cu) (net 14))
+  (segment (start 180.55 98) (end 182.425 96.125) (width 1) (layer B.Cu) (net 14))
+  (segment (start 182.425 90.825) (end 178 86.4) (width 1) (layer B.Cu) (net 14))
+  (segment (start 182.425 96.125) (end 182.425 90.825) (width 1) (layer B.Cu) (net 14))
+  (segment (start 178 62.5) (end 178 86.4) (width 1) (layer B.Cu) (net 14))
   (segment (start 174.5 90.75) (end 174.25 91) (width 2) (layer B.Cu) (net 15))
   (segment (start 172.4271 92.8229) (end 174.5 90.75) (width 2) (layer B.Cu) (net 15))
@@
   (segment (start 170.75 33.75) (end 170.75 34) (width 2) (layer B.Cu) (net 15))
   (segment (start 170.75 34) (end 174.75 38) (width 2) (layer B.Cu) (net 15))
-  (segment (start 142.5 33.76) (end 160.26 33.76) (width 2) (layer B.Cu) (net 16))
-  (segment (start 160.26 33.76) (end 164.5 38) (width 2) (layer B.Cu) (net 16))
-  (segment (start 160.27 33.75) (end 160.26 33.76) (width 2) (layer B.Cu) (net 16))
-  (segment (start 168.21 33.75) (end 160.27 33.75) (width 2) (layer B.Cu) (net 16))
+  (segment (start 153.75 48.75) (end 164.5 38) (width 2) (layer B.Cu) (net 16))
+  (segment (start 153.75 49) (end 153.75 48.75) (width 2) (layer B.Cu) (net 16))
+  (segment (start 164.5 37.46) (end 168.21 33.75) (width 2) (layer B.Cu) (net 16))
+  (segment (start 164.5 38) (end 164.5 37.46) (width 2) (layer B.Cu) (net 16))
 )
