File: Flyback/Flyback.sch (KiCad schematic (older format))
At the start: 53 parts, among them Q1 IRF840, U1 UC3843_DIP8

Commit message: PCB_v0
Parts:
- added RL1: 68 2W, Flyback:RCarga30mm, symbol Device:R
- CIN2: footprint Capacitor_THT:C_Axial_L3.8mm_D2.6mm_P10.00mm_Horizontal -> Capacitor_THT:C_Axial_L3.8mm_D2.6mm_P12.50mm_Horizontal
- CMASAS1: footprint Capacitor_THT:C_Disc_D6.0mm_W2.5mm_P5.00mm -> Capacitor_THT:C_Rect_L9.0mm_W3.2mm_P7.50mm_MKT
- CREG1: footprint Capacitor_THT:C_Disc_D3.8mm_W2.6mm_P2.50mm -> Capacitor_THT:C_Rect_L7.2mm_W2.5mm_P5.00mm_FKS2_FKP2_MKS2_MKP2
- DB1: footprint Diode_THT:Diode_Bridge_Round_D9.8mm -> Flyback:PuenteDiodos
- DF2: footprint Diode_THT:D_DO-41_SOD81_P10.16mm_Horizontal -> Diode_THT:D_DO-41_SOD81_P12.70mm_Horizontal
- DREG1: footprint Package_TO_SOT_THT:TO-92L_Wide -> Package_TO_SOT_THT:TO-92L_Inline_Wide
- RFB1, RFB2, RPOL-REG1: footprint Resistor_THT:R_Axial_DIN0207_L6.3mm_D2.5mm_P10.16mm_Horizontal -> Resistor_THT:R_Axial_DIN0309_L9.0mm_D3.2mm_P15.24mm_Horizontal
- RG1: value 22 1/4W -> 10 1/4W
- RPOL-DF2: footprint Resistor_THT:R_Axial_DIN0207_L6.3mm_D2.5mm_P10.16mm_Horizontal -> Flyback:R12,5
- RSENSE1: value 3.3 3W -> 0.5 3W
Connections:
- net GNDREF: now also RL1.1
- net I-IN-: now also DB1.2 (~~); no longer DB1.4 (~~)
- net ID-: now also RL1.2
- net at TH1.1: now also DB1.4 (~~); no longer DB1.2 (~~)
Other:
- moved on the sheet: F1, JGND1, JN1, JOUT1, JV1, TH1
Changed lines of the file:
@@
 L Device:Thermistor_NTC TH1
 U 1 1 5D910C56
-P 1700 2450
-F 0 "TH1" V 1850 2350 50  0000 L CNN
-F 1 "Thermistor_NTC" V 1950 2350 50  0000 L CNN
-F 2 "Resistor_THT:R_Axial_DIN0207_L6.3mm_D2.5mm_P2.54mm_Vertical" H 1700 2500 50  0001 C CNN
-F 3 "~" H 1700 2500 50  0001 C CNN
-	1    1700 2450
+P 1250 2450
+F 0 "TH1" V 1400 2350 50  0000 L CNN
+F 1 "Thermistor_NTC" V 1500 2350 50  0000 L CNN
+F 2 "Resistor_THT:R_Axial_DIN0207_L6.3mm_D2.5mm_P2.54mm_Vertical" H 1250 2500 50  0001 C CNN
+F 3 "~" H 1250 2500 50  0001 C CNN
+	1    1250 2450
 	0    1    1    0
 $EndComp
@@
 F 0 "CIN2" H 4215 1596 50  0000 L CNN
 F 1 "0.1u 400V" H 4215 1505 50  0000 L CNN
-F 2 "Capacitor_THT:C_Axial_L3.8mm_D2.6mm_P10.00mm_Horizontal" H 4138 1400 50  0001 C CNN
+F 2 "Capacitor_THT:C_Axial_L3.8mm_D2.6mm_P12.50mm_Horizontal" H 4138 1400 50  0001 C CNN
 F 3 "~" H 4100 1550 50  0001 C CNN
 	1    4100 1550
@@
 L Connector:Conn_01x01_Male JV1
 U 1 1 5D9135EC
-P 850 1550
-F 0 "JV1" H 950 1500 50  0000 L CNN
-F 1 "AC" H 950 1400 50  0000 L CNN
-F 2 "Connector:Banana_Jack_1Pin" H 850 1550 50  0001 C CNN
-F 3 "~" H 850 1550 50  0001 C CNN
-	1    850  1550
+P 650 1550
+F 0 "JV1" H 750 1500 50  0000 L CNN
+F 1 "AC" H 750 1400 50  0000 L CNN
+F 2 "Connector:Banana_Jack_1Pin" H 650 1550 50  0001 C CNN
+F 3 "~" H 650 1550 50  0001 C CNN
+	1    650  1550
 	1    0    0    -1
 $EndComp
@@
 L Connector:Conn_01x01_Male JN1
 U 1 1 5D913E61
-P 850 2450
-F 0 "JN1" H 950 2400 50  0000 L CNN
-F 1 "AC" H 950 2300 50  0000 L CNN
-F 2 "Connector:Banana_Jack_1Pin" H 850 2450 50  0001 C CNN
-F 3 "~" H 850 2450 50  0001 C CNN
-	1    850  2450
+P 650 2450
+F 0 "JN1" H 750 2400 50  0000 L CNN
+F 1 "AC" H 750 2300 50  0000 L CNN
+F 2 "Connector:Banana_Jack_1Pin" H 650 2450 50  0001 C CNN
+F 3 "~" H 650 2450 50  0001 C CNN
+	1    650  2450
 	1    0    0    -1
 $EndComp
@@
 F 0 "RPOL-DF2" H 3050 2950 50  0000 L CNN
 F 1 "220k 1W" H 3050 2850 50  0000 L CNN
-F 2 "Resistor_THT:R_Axial_DIN0207_L6.3mm_D2.5mm_P10.16mm_Horizontal" V 2880 2900 50  0001 C CNN
+F 2 "Flyback:R12,5" V 2880 2900 50  0001 C CNN
 F 3 "~" H 2950 2900 50  0001 C CNN
 	1    2950 2900
@@
 $EndComp
 $Comp
-L Diode_Bridge:W10G DB1
-U 1 1 5D915B82
-P 2250 1550
-F 0 "DB1" V 2500 1150 50  0000 L CNN
-F 1 "W10G" V 2400 1300 50  0000 R CNN
-F 2 "Diode_THT:Diode_Bridge_Round_D9.8mm" H 2400 1675 50  0001 L CNN
-F 3 "https://www.vishay.com/docs/88769/woo5g.pdf" H 2250 1550 50  0001 C CNN
-	1    2250 1550
-	0    -1   -1   0
-$EndComp
-$Comp
 L Transistor_FET:IRF740 Q1
 U 1 1 5D917572
@@
 F 0 "DF2" H 3700 3466 50  0000 C CNN
 F 1 "UF4007" H 3700 3375 50  0000 C CNN
-F 2 "Diode_THT:D_DO-41_SOD81_P10.16mm_Horizontal" H 3700 3075 50  0001 C CNN
+F 2 "Diode_THT:D_DO-41_SOD81_P12.70mm_Horizontal" H 3700 3075 50  0001 C CNN
 F 3 "http://diotec.com/tl_files/diotec/files/pdf/datasheets/ba157" H 3700 3250 50  0001 C CNN
 	1    3700 3250
@@
 P 4400 4250
 F 0 "RG1" V 4150 4250 50  0000 R CNN
-F 1 "22 1/4W" V 4250 4150 50  0000 L CNN
+F 1 "10 1/4W" V 4250 4150 50  0000 L CNN
 F 2 "Resistor_THT:R_Axial_DIN0207_L6.3mm_D2.5mm_P10.16mm_Horizontal" V 4330 4250 50  0001 C CNN
 F 3 "~" H 4400 4250 50  0001 C CNN
@@
 F 0 "DREG1" V 8100 4200 50  0000 R CNN
 F 1 "TL431LP" V 8000 4200 50  0000 R CNN
-F 2 "Package_TO_SOT_THT:TO-92L_Wide" H 8050 4150 50  0001 C CIN
+F 2 "Package_TO_SOT_THT:TO-92L_Inline_Wide" H 8050 4150 50  0001 C CIN
 F 3 "http://www.ti.com/lit/ds/symlink/tl431.pdf" H 8050 4300 50  0001 C CIN
 	1    8050 4300
@@
 P 5550 5250
 F 0 "RSENSE1" H 5450 5300 50  0000 R CNN
-F 1 "3.3 3W" H 5450 5200 50  0000 R CNN
+F 1 "0.5 3W" H 5450 5200 50  0000 R CNN
 F 2 "Resistor_THT:R_Axial_DIN0309_L9.0mm_D3.2mm_P15.24mm_Horizontal" V 5480 5250 50  0001 C CNN
 F 3 "~" H 5550 5250 50  0001 C CNN
@@
 F 0 "RPOL-REG1" V 7700 4100 50  0000 R CNN
 F 1 "100 1/4W" V 7600 4100 50  0000 R CNN
-F 2 "Resistor_THT:R_Axial_DIN0207_L6.3mm_D2.5mm_P10.16mm_Horizontal" V 7430 4000 50  0001 C CNN
+F 2 "Resistor_THT:R_Axial_DIN0309_L9.0mm_D3.2mm_P15.24mm_Horizontal" V 7430 4000 50  0001 C CNN
 F 3 "~" H 7500 4000 50  0001 C CNN
 	1    7500 4000
@@
 $EndComp
 Wire Wire Line
-	2250 1250 2250 1000
-Wire Wire Line
-	2750 1550 2550 1550
-Wire Wire Line
 	2750 1550 2750 2450
 Wire Wire Line
@@
 F 0 "CREG1" V 8650 4100 50  0000 R CNN
 F 1 "10n" V 8550 4100 50  0000 R CNN
-F 2 "Capacitor_THT:C_Disc_D3.8mm_W2.6mm_P2.50mm" H 8438 3850 50  0001 C CNN
+F 2 "Capacitor_THT:C_Rect_L7.2mm_W2.5mm_P5.00mm_FKS2_FKP2_MKS2_MKP2" H 8438 3850 50  0001 C CNN
 F 3 "~" H 8400 4000 50  0001 C CNN
 	1    8400 4000
@@
 L Connector:Conn_01x01_Male JOUT1
 U 1 1 5DA45919
-P 10700 1250
-F 0 "JOUT1" H 10900 1350 50  0000 R CNN
-F 1 "OUT+" H 10900 1450 50  0000 R CNN
-F 2 "Connector:Banana_Jack_1Pin" H 10700 1250 50  0001 C CNN
-F 3 "~" H 10700 1250 50  0001 C CNN
-	1    10700 1250
+P 11000 1250
+F 0 "JOUT1" H 11200 1350 50  0000 R CNN
+F 1 "OUT+" H 11200 1450 50  0000 R CNN
+F 2 "Connector:Banana_Jack_1Pin" H 11000 1250 50  0001 C CNN
+F 3 "~" H 11000 1250 50  0001 C CNN
+	1    11000 1250
 	-1   0    0    1
 $EndComp
@@
 L Connector:Conn_01x01_Male JGND1
 U 1 1 5DA709B0
-P 10700 2100
-F 0 "JGND1" H 10900 2200 50  0000 R CNN
-F 1 "OUT-" H 10900 2300 50  0000 R CNN
-F 2 "Connector:Banana_Jack_1Pin" H 10700 2100 50  0001 C CNN
-F 3 "~" H 10700 2100 50  0001 C CNN
-	1    10700 2100
+P 11000 2100
+F 0 "JGND1" H 11200 2200 50  0000 R CNN
+F 1 "OUT-" H 11200 2300 50  0000 R CNN
+F 2 "Connector:Banana_Jack_1Pin" H 11000 2100 50  0001 C CNN
+F 3 "~" H 11000 2100 50  0001 C CNN
+	1    11000 2100
 	-1   0    0    1
 $EndComp
@@
 Wire Wire Line
 	9450 1700 9450 1750
-$Comp
-L power:GNDREF #PWR0119
-U 1 1 5DA0BD19
-P 10100 2150
-F 0 "#PWR0119" H 10100 1900 50  0001 C CNN
-F 1 "GNDREF" H 10100 2000 50  0000 C CNN
-F 2 "" H 10100 2150 50  0001 C CNN
-F 3 "" H 10100 2150 50  0001 C CNN
-	1    10100 2150
-	1    0    0    -1
-$EndComp
 $Comp
 L Device:LED DLED1
@@
 Wire Wire Line
 	8850 1250 9150 1250
-Connection ~ 9450 1250
-Wire Wire Line
-	10500 2100 10100 2100
-Wire Wire Line
-	10100 2100 10100 2150
 Connection ~ 9150 1250
 Wire Wire Line
@@
 F 0 "RFB1" H 9050 4200 50  0000 R CNN
 F 1 "3.3k 1/4W" H 9050 4300 50  0000 R CNN
-F 2 "Resistor_THT:R_Axial_DIN0207_L6.3mm_D2.5mm_P10.16mm_Horizontal" V 9080 4250 50  0001 C CNN
+F 2 "Resistor_THT:R_Axial_DIN0309_L9.0mm_D3.2mm_P15.24mm_Horizontal" V 9080 4250 50  0001 C CNN
 F 3 "~" H 9150 4250 50  0001 C CNN
 	1    9150 4250
@@
 F 0 "RFB2" H 9050 3700 50  0000 R CNN
 F 1 "2.7k 1/4W" H 9050 3800 50  0000 R CNN
-F 2 "Resistor_THT:R_Axial_DIN0207_L6.3mm_D2.5mm_P10.16mm_Horizontal" V 9080 3750 50  0001 C CNN
+F 2 "Resistor_THT:R_Axial_DIN0309_L9.0mm_D3.2mm_P15.24mm_Horizontal" V 9080 3750 50  0001 C CNN
 F 3 "~" H 9150 3750 50  0001 C CNN
 	1    9150 3750
@@
 Wire Wire Line
 	1650 1450 1650 1550
-Wire Wire Line
-	1800 1450 1800 1550
-Wire Wire Line
-	1800 1550 1950 1550
 Wire Wire Line
 	9150 1150 9150 1250
@@
 	2250 1000 2550 1000
 Wire Wire Line
-	1050 2450 1550 2450
-Wire Wire Line
-	1850 2450 2750 2450
-Wire Wire Line
 	2500 5050 2500 5100
 Connection ~ 2500 5050
@@
 F 0 "CMASAS1" V 7000 5450 50  0000 R CNN
 F 1 "4.7n 2000V" V 6900 5450 50  0000 R CNN
-F 2 "Capacitor_THT:C_Disc_D6.0mm_W2.5mm_P5.00mm" H 6788 5200 50  0001 C CNN
+F 2 "Capacitor_THT:C_Rect_L9.0mm_W3.2mm_P7.50mm_MKT" H 6788 5200 50  0001 C CNN
 F 3 "~" H 6750 5350 50  0001 C CNN
 	1    6750 5350
@@
 Wire Wire Line
 	7100 5350 7100 5500
-Wire Wire Line
-	9450 1250 10500 1250
 $Comp
 L Device:Fuse F1
 U 1 1 5D9966CE
-P 1350 1550
-F 0 "F1" V 1153 1550 50  0000 C CNN
-F 1 "250V 1A" V 1244 1550 50  0000 C CNN
-F 2 "Fuse:Fuseholder_Cylinder-5x20mm_Stelvio-Kontek_PTF78_Horizontal_Open" V 1280 1550 50  0001 C CNN
-F 3 "~" H 1350 1550 50  0001 C CNN
-	1    1350 1550
+P 1250 1550
+F 0 "F1" V 1053 1550 50  0000 C CNN
+F 1 "250V 1A" V 1144 1550 50  0000 C CNN
+F 2 "Fuse:Fuseholder_Cylinder-5x20mm_Stelvio-Kontek_PTF78_Horizontal_Open" V 1180 1550 50  0001 C CNN
+F 3 "~" H 1250 1550 50  0001 C CNN
+	1    1250 1550
 	0    1    1    0
 $EndComp
-Wire Wire Line
-	1500 1550 1650 1550
-Wire Wire Line
-	1050 1550 1200 1550
+Connection ~ 9450 1250
+$Comp
+L power:GNDREF #PWR0123
+U 1 1 5D9EBFDA
+P 10100 2150
+F 0 "#PWR0123" H 10100 1900 50  0001 C CNN
+F 1 "GNDREF" H 10100 2000 50  0000 C CNN
+F 2 "" H 10100 2150 50  0001 C CNN
+F 3 "" H 10100 2150 50  0001 C CNN
+	1    10100 2150
+	1    0    0    -1
+$EndComp
+Wire Wire Line
+	10100 1700 10100 2150
+$Comp
+L Device:R RL1
+U 1 1 5D9E2A2B
+P 10100 1550
+F 0 "RL1" H 10000 1500 50  0000 R CNN
+F 1 "68 2W" H 10000 1600 50  0000 R CNN
+F 2 "Flyback:RCarga30mm" V 10030 1550 50  0001 C CNN
+F 3 "~" H 10100 1550 50  0001 C CNN
+	1    10100 1550
+	-1   0    0    1
+$EndComp
+Wire Wire Line
+	10100 1400 10100 1250
+Connection ~ 10100 1250
+Wire Wire Line
+	10800 2100 10550 2100
+Wire Wire Line
+	10550 2100 10550 2150
+Wire Wire Line
+	1400 1550 1650 1550
+Wire Wire Line
+	1400 2450 2750 2450
+Wire Wire Line
+	10100 1250 10800 1250
+Wire Wire Line
+	10000 1250 10100 1250
+Wire Wire Line
+	9450 1250 10100 1250
+$Comp
+L power:GNDREF #PWR0119
+U 1 1 5DB41863
+P 10550 2150
+F 0 "#PWR0119" H 10550 1900 50  0001 C CNN
+F 1 "GNDREF" H 10550 2000 50  0000 C CNN
+F 2 "" H 10550 2150 50  0001 C CNN
+F 3 "" H 10550 2150 50  0001 C CNN
+	1    10550 2150
+	1    0    0    -1
+$EndComp
+Wire Wire Line
+	850  1550 1100 1550
+Wire Wire Line
+	850  2450 1100 2450
+Wire Wire Line
+	1800 1450 1800 1550
+Wire Wire Line
+	2250 1250 2250 1000
+$Comp
+L Diode_Bridge:W10G DB1
+U 1 1 5D915B82
+P 2250 1550
+F 0 "DB1" V 2500 1150 50  0000 L CNN
+F 1 "W10G" V 2400 1300 50  0000 R CNN
+F 2 "Flyback:PuenteDiodos" H 2400 1675 50  0001 L CNN
+F 3 "https://www.vishay.com/docs/88769/woo5g.pdf" H 2250 1550 50  0001 C CNN
+	1    2250 1550
+	0    1    -1   0
+$EndComp
+Wire Wire Line
+	2750 1550 2550 1550
+Wire Wire Line
+	1800 1550 1950 1550
 $EndSCHEMATC
