File: Flyback/_saved_Flyback.sch (KiCad schematic (older format))
At the start: 54 parts, among them Q1 IRF840, U1 UC3843_DIP8

Commit message: agrandado la Rsense de 3W a 20.32mm de largo y retoques minimos
Parts:
- RSENSE1: footprint Resistor_THT:R_Axial_DIN0309_L9.0mm_D3.2mm_P15.24mm_Horizontal -> Resistor_THT:R_Axial_DIN0411_L9.9mm_D3.6mm_P20.32mm_Horizontal
Changed lines of the file:
@@
 F 0 "RSENSE1" H 5450 5300 50  0000 R CNN
 F 1 "0.5 3W" H 5450 5200 50  0000 R CNN
-F 2 "Resistor_THT:R_Axial_DIN0309_L9.0mm_D3.2mm_P15.24mm_Horizontal" V 5480 5250 50  0001 C CNN
+F 2 "Resistor_THT:R_Axial_DIN0411_L9.9mm_D3.6mm_P20.32mm_Horizontal" V 5480 5250 50  0001 C CNN
 F 3 "~" H 5550 5250 50  0001 C CNN
 	1    5550 5250
